File: STLinkV2.1.kicad_sch (KiCad schematic)
At the start: 53 parts, among them J1 USB_C_USB2.0, J2 SWD, J3 USB_A, Q1 S8050, U1 RT9193-18GB, U2 USBLC6-2SC6, U3 STM32F103CBTx, Y1 8MHz

Commit message: Change board size and output connector.
Parts:
- removed J2: SWD, Conn_02x05_Horizontal_2Layer:Conn_02x05_Horizontal_2Layer, symbol Connector_Generic:Conn_02x05_Counter_Clockwise
- removed R11, R7: 100, Resistor_SMD:R_0603_1608Metric, symbol Device:R_Small
- added J2: SWD, Conn_Horizontal_2Layer:Conn_02x04_Horizontal_2Layer, symbol Connector_Generic:Conn_02x04_Counter_Clockwise
Connections:
- net +3.3V: now also J2.1 (Pin_1)
- net +5V: now also J2.8 (Pin_8)
- net GND: now also J2.2 (Pin_2), J2.7 (Pin_7)
- net ST_RX: now also J2.6 (Pin_6)
- net ST_TX: now also J2.5 (Pin_5)
- net at R6.2: now also J2.4 (Pin_4)
- net at R5.2: now also J2.3 (Pin_3)
- net O_RST: no longer names the net of U3.18 (PB0)
- net O_SWO: no longer names the net of U3.31 (PA10)
- no-connect marks 21 -> 23
